File: hardware/pcb/Dumber/dumber-v3/dumber-v3.kicad_sch (KiCad schematic)
At the start: 0 parts

Commit message: correction de bugs lorsque le watchdog est actif ainsi que les moteurs + bug lorsque la batterie est faible
Other:
- title: (none) -> Dumber-3
Changed lines of the file:
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@@
   (paper "A4")
   (title_block
+    (title "Dumber-3")
     (date "2022-06-08")
-    (rev "1.0")
+    (rev "2.2")
     (company "INSA - GEI")
   )
